File: fistion.kicad_pcb (KiCad board)
At the start: 2 copper layers, 165 x 92.1 mm, 67 parts, among them J1 Conn_01x07, J2 Conn_01x07, J3 Conn_01x04, U1 nice_nano, U2 MT25QL128ABA1ESE

Commit message: Pending
Parts:
- removed KEY15: SW_Push, lib:Kailh_PG1232
- removed the KEY6 at (169.0, 52.0)
- removed the REF** at (106.0, 71.5)
- removed the REF** at (99.0, 75.5)
- removed the REF** at (99.0, 73.5)
- removed the REF** at (99.0, 76.5)
- removed the REF** at (99.0, 70.5)
- removed the REF** at (99.0, 71.5)
- removed the REF** at (99.0, 69.5)
- removed the REF** at (99.0, 72.5)
- removed the REF** at (103.0, 108.5)
- removed the REF** at (103.0, 107.5)
- removed the REF** at (103.0, 109.5)
- removed the REF** at (106.0, 70.5)
- removed the REF** at (103.0, 106.5)
- removed the REF** at (99.0, 107.5)
- removed the REF** at (99.0, 108.5)
- removed the REF** at (99.0, 106.5)
- removed the REF** at (99.0, 109.5)
- removed the REF** at (70.0, 32.0)
- removed the REF** at (70.0, 31.0)
- removed the REF** at (70.0, 33.0)
- removed the REF** at (70.0, 30.0)
- removed the REF** at (67.0, 31.0)
- removed the REF** at (106.0, 72.5)
- removed the REF** at (67.0, 32.0)
- removed the REF** at (67.0, 30.0)
- removed the REF** at (67.0, 33.0)
- removed the REF** at (70.0, 50.0)
- removed the REF** at (70.0, 49.0)
- removed the REF** at (70.0, 51.0)
- removed the REF** at (70.0, 48.0)
- removed the REF** at (67.0, 49.0)
- removed the REF** at (67.0, 50.0)
- removed the REF** at (67.0, 48.0)
- removed the REF** at (106.0, 69.5)
- removed the REF** at (67.0, 51.0)
- removed the REF** at (106.0, 75.5)
- removed the REF** at (106.0, 74.5)
- removed the REF** at (106.0, 76.5)
- removed the REF** at (106.0, 73.5)
- removed the REF** at (99.0, 74.5)
- removed palm1: Conn_01x04, fistion:palm-female
- removed palm2: Conn_01x04, fistion:palm-male
- added J4: Conn_01x02, Connector_PinSocket_2.54mm:PinSocket_1x02_P2.54mm_Vertical, F.Cu at (150.5, 100.1)
- added KEY11: SW_Push, lib:Kailh_PG1232, F.Cu at (115.0, 64.0)
- added REF**: PinHeader_1x05_P2.54mm_Vertical, Connector_PinHeader_2.54mm:PinHeader_1x05_P2.54mm_Vertical, F.Cu at (98.9, 84.2)
- added REF**: breakaway-mousebites, Keebio-Parts:breakaway-mousebites, F.Cu at (105.5, 74.1)
- added REF**: breakaway-mousebites, Keebio-Parts:breakaway-mousebites, F.Cu at (105.5, 67.7)
- added REF**: breakaway-mousebites, Keebio-Parts:breakaway-mousebites, F.Cu at (109.2, 111.0)
- added REF**: breakaway-mousebites, Keebio-Parts:breakaway-mousebites, F.Cu at (156.8, 111.0)
- added REF**: palm-conn, fistion:palm-conn, F.Cu at (133.5, 113.6)
- added REF**: palm-conn, fistion:palm-conn, F.Cu at (133.5, 108.0)
- J1: value Conn_01x07 -> Conn_01x04; footprint fistion:thumb-male -> steno:OLED
- J2: value Conn_01x07 -> Conn_01x06; footprint fistion:thumb-female -> fistion:thumb-thumb
- J3: value Conn_01x04 -> Conn_01x06; footprint steno:OLED -> fistion:thumb-palm
- PUSH1: renamed from PUSH2; footprint Button_Switch_SMD:SW_SPST_B3U-1000P -> Button_Switch_SMD:SW_SPST_EVQQ2
- PUSH2: renamed from PUSH1; footprint Button_Switch_SMD:SW_SPST_B3U-1000P -> Button_Switch_SMD:SW_SPST_EVQQ2
- R3: renamed from R1; moved to B.Cu
- U2: moved to B.Cu
- moved J3 96.5 mm to (108.0, 92.5), turned to 90 degrees
- moved KEY14 72.6 mm to (96.5, 71.8)
- moved KEY13 70.0 mm to (78.5, 69.8)
- moved J2 62.6 mm to (96.7, 91.0), turned to 111.3 degrees
- moved R3 44.0 mm to (119.5, 91.0), turned to 90 degrees
- moved U2 39.0 mm to (123.6, 88.4), turned to 270 degrees
- moved J1 36.4 mm to (72.7, 71.8), turned to 309 degrees
- moved KEY12 36.0 mm to (133.0, 69.0)
- moved PUSH1 23.8 mm to (150.9, 87.4)
- moved PUSH2 23.8 mm to (150.9, 87.4), turned to 180 degrees
- moved R1 17.0 mm to (150.0, 92.4)
- moved R2 17.0 mm to (150.0, 92.4)
- moved U1 16.0 mm to (142.0, 87.5)
- moved KEY1 3.00 mm to (79.0, 37.0)
- moved KEY10 3.00 mm to (151.0, 72.0)
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- renumbered KEY11 to KEY10, KEY7 to KEY6, KEY8 to KEY7, KEY9 to KEY8, KEY10 to KEY9, R2 to R1, R3 to R2
Connections:
- J1 pad 1: GND -> thumb_gnd
- J1 pad 2: R3C1 -> thumb_vcc
- J1 pad 3: R3C2 -> thumb_scl
- J1 pad 4: R3C3 -> thumb_sda
- J2 pad 2: thumb_R3C1 -> thumb_vcc
- J2 pad 3: thumb_R3C2 -> thumb_sda
- J2 pad 4: thumb_R3C3 -> thumb_scl
- J2 pad 5: thumb_vcc -> thumb_R3C1
- J2 pad 6: thumb_scl -> thumb_R3C2
- J3 pad 1: thumb_gnd -> GND
- J3 pad 2: thumb_vcc -> 3V3
- J3 pad 3: thumb_scl -> SDA
- J3 pad 4: thumb_sda -> SCL
- KEY12 pad 2: R2C6 -> R3C4
- U1 pad 10: R1C6 -> R1C5
- U1 pad 11: R2C5 -> R2C4
- U1 pad 12: R1C5 -> R3C4
- U1 pad 13: R2C1 -> R2C2
- U1 pad 14: R1C1 -> R2C1
- U1 pad 15: R2C2 -> R3C3
- U1 pad 16: R1C2 -> R1C1
- U1 pad 17: R2C3 -> R1C2
- U1 pad 18: R1C3 -> R2C3
- U1 pad 19: R2C4 -> R1C3
- U1 pad 20: R1C4 -> Net-(U1-Pad20)
- U1 pad 24: Net-(U1-Pad24) -> BAT
- U1 pad 31: R3C3 -> R1C4
- U1 pad 5: SCLK -> MOSI
- U1 pad 6: MOSI -> SCLK
- U1 pad 7: CS -> MISO
- U1 pad 8: MISO -> CS
- U1 pad 9: R2C6 -> R2C5
Routing:
- net 3V3: track 89.3 -> 51.3 mm
- net R1C6: track 36.3 -> 0.00 mm
- net R3C2: track 50.4 -> 26.0 mm
- net thumb_R3C1: track 45.7 -> 22.2 mm
- net R3C1: track 51.0 -> 28.0 mm
- net R1C4: track 76.4 -> 54.0 mm
- net thumb_R3C2: track 30.7 -> 9.08 mm
- net R2C4: track 57.6 -> 36.1 mm
- net R2C6: track 21.4 -> 0.00 mm
- net CS: track 5.61 -> 26.8 mm
- net thumb_vcc: track 23.8 -> 42.8 mm
- net MISO: track 8.40 -> 27.2 mm
- net SCLK: track 9.60 -> 25.4 mm
- net thumb_R3C3: track 15.5 -> 0.00 mm
- net thumb_sda: track 21.1 -> 35.1 mm
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Other:
- board size 165 x 92.1 mm -> 96.6 x 154.8 mm

Commit message: backup
Parts:
- removed KEY1, KEY6: SW_Push, lib:Kailh_PG1232
- removed the REF** at (98.9, 84.2)
- removed the REF** at (105.5, 74.1)
- removed the REF** at (105.5, 67.7)
- removed the REF** at (133.5, 113.6)
- removed the REF** at (133.5, 108.0)
- added REF**: breakaway-hole-big, Keebio-Parts:breakaway-hole-big, F.Cu at (105.5, 79.6)
- added REF**: breakaway-mousebites, Keebio-Parts:breakaway-mousebites, F.Cu at (105.5, 75.8)
- added REF**: breakaway-mousebites, Keebio-Parts:breakaway-mousebites, F.Cu at (105.5, 69.5)
- J4: footprint Connector_PinSocket_2.54mm:PinSocket_1x02_P2.54mm_Vertical -> Connector_PinHeader_2.54mm:PinHeader_1x02_P2.54mm_Vertical
- KEY10, KEY11, KEY12, KEY13, KEY14, KEY2, KEY3, KEY4, KEY5, KEY8, KEY9: footprint lib:Kailh_PG1232 -> Keebio-Parts:Kailh-PG1350-1u-reversible-No-Clickhole
- KEY7: footprint lib:Kailh_PG1232 -> Keebio-Parts:Kailh-PG1350-1u-reversible-No-Clickhole; moved to B.Cu
- moved J1 17.1 mm to (78.0, 55.5), turned to 90 degrees
- moved U2 14.4 mm to (138.0, 87.5), turned to 90 degrees
- moved R3 14.0 mm to (133.5, 91.0), turned to 270 degrees
- moved KEY11 8.50 mm to (115.0, 55.5), turned to 180 degrees
- moved KEY12 8.50 mm to (133.0, 60.5), turned to 180 degrees
- moved KEY3 8.50 mm to (115.0, 21.5), turned to 180 degrees
- moved KEY4 8.50 mm to (133.0, 26.5), turned to 180 degrees
- moved KEY8 8.50 mm to (115.0, 38.5), turned to 180 degrees
- moved KEY9 8.50 mm to (133.0, 43.5), turned to 180 degrees
- moved J2 1.84 mm to (97.2, 92.8), turned to 113 degrees
- moved KEY13 1.70 mm to (78.5, 71.5), turned to 180 degrees
- moved KEY14 1.60 mm to (96.5, 73.4), turned to 180 degrees
- moved J3 1.00 mm to (107.0, 92.5)
- moved KEY10 1.00 mm to (151.0, 71.0), turned to 180 degrees
- moved KEY5 1.00 mm to (151.0, 54.0), turned to 180 degrees
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Connections:
- J1 pad 1: thumb_gnd -> GND
- J1 pad 2: thumb_vcc -> 3V3
- J1 pad 3: thumb_scl -> SCL
- J1 pad 4: thumb_sda -> SDA
- U1 pad 11: R2C4 -> R3C4
- U1 pad 12: R3C4 -> R2C4
- U1 pad 14: R2C1 -> R1C2
- U1 pad 16: R1C1 -> R2C3
- U1 pad 17: R1C2 -> R1C3
- U1 pad 18: R2C3 -> Net-(U1-Pad18)
- U1 pad 19: R1C3 -> Net-(U1-Pad19)
- U1 pad 5: MOSI -> CS
- U1 pad 6: SCLK -> MISO
- U1 pad 7: MISO -> SCLK
- U1 pad 8: CS -> MOSI
Routing:
- net GND: track 9.10 -> 319.1 mm, vias 3 -> 1
- net 3V3: track 51.3 -> 151.3 mm
- net R2C1: track 97.8 -> 0.00 mm
- net R1C1: track 95.8 -> 0.00 mm
- net thumb_gnd: track 0.00 -> 56.7 mm
- net SDA: track 69.4 -> 117.7 mm, vias 0 -> 1
- net thumb_vcc: track 42.8 -> 0.00 mm
- net SCL: track 70.8 -> 107.1 mm, vias 0 -> 1
- net thumb_sda: track 35.1 -> 0.03 mm
- net thumb_scl: track 31.4 -> 0.00 mm
- net R3C4: track 10.7 -> 34.3 mm
- net R1C4: track 54.0 -> 77.4 mm
- net R3C3: track 36.4 -> 58.9 mm
- net MOSI: track 25.3 -> 4.87 mm
- net SCLK: track 25.4 -> 5.39 mm
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- removed copper zone on B.Cu, net GND
- removed copper zone on F.Cu, net GND
- removed copper zone on B.Cu, net thumb_gnd
- removed copper zone on F.Cu, net thumb_gnd
Other:
- board size 96.6 x 154.8 mm -> 90.5 x 147.9 mm

Commit message: new start
Parts:
- removed J3: Conn_01x06, fistion:thumb-palm
- removed J4: Conn_01x02, Connector_PinHeader_2.54mm:PinHeader_1x02_P2.54mm_Vertical
- removed KEY10, KEY11, KEY12, KEY13, KEY14, KEY2, KEY3, KEY4, KEY5, KEY7, KEY8, KEY9: SW_Push, Keebio-Parts:Kailh-PG1350-1u-reversible-No-Clickhole
- removed PUSH1, PUSH2: SW_Push, Button_Switch_SMD:SW_SPST_EVQQ2
- removed the REF** at (105.5, 79.6)
- removed the REF** at (109.2, 111.0)
- removed the REF** at (156.8, 111.0)
- removed the REF** at (105.5, 75.8)
- removed the REF** at (105.5, 69.5)
- added C1: 10nF, Capacitor_SMD:C_0603_1608Metric, F.Cu at (222.2, 54.8)
- added C2: 4.7uF, Capacitor_SMD:C_0603_1608Metric, F.Cu at (199.8, 93.3)
- added C3: 0.1uF, Capacitor_SMD:C_0603_1608Metric, F.Cu at (192.1, 60.5)
- added C4: Li Cap, Capacitor_THT:CP_Radial_D13.0mm_P5.00mm, F.Cu at (174.7, 66.5)
- added C5: 4.7uF, Capacitor_SMD:C_0603_1608Metric, F.Cu at (184.5, 21.2)
- added C6: 10nF, Capacitor_SMD:C_0603_1608Metric, F.Cu at (187.5, 24.2)
- added C7: 0.1uF, Capacitor_SMD:C_0603_1608Metric, F.Cu at (191.8, 17.4)
- added C8: 47uF, Capacitor_SMD:C_0805_2012Metric, F.Cu at (193.5, 17.4)
- added D1: D_Small, Diode_SMD:D_SOD-123, F.Cu at (231.3, 71.5)
- added D2: LED_RABG, LED_SMD:LED_ASMB-KTF0-0A306, F.Cu at (211.7, 71.9)
- added D3: D, Diode_SMD:D_SOD-123, F.Cu at (215.9, 110.4)
- added JP1: All or none, Jumper:SolderJumper-3_P1.3mm_Open_RoundedPad1.0x1.5mm, F.Cu at (172.3, 80.2)
- added JP2: SolderJumper_3_Open, Jumper:SolderJumper-3_P1.3mm_Open_RoundedPad1.0x1.5mm, F.Cu at (187.2, 61.0)
- added JP3: ~, Jumper:SolderJumper-2_P1.3mm_Open_RoundedPad1.0x1.5mm, F.Cu at (197.2, 26.1)
- added JP4: SolderJumper_2_Open, Jumper:SolderJumper-2_P1.3mm_Open_RoundedPad1.0x1.5mm, F.Cu at (196.7, 19.6)
- added K1: diode-choc, pg1232:pg1232-DCR, F.Cu at (103.4, 42.1)
- added K10: diode-choc, pg1232:pg1232-DC, F.Cu at (121.4, 60.1)
- added K11: diode-choc, pg1232:pg1232-DCL, F.Cu at (139.4, 67.1)
- added K12: diode-choc, pg1232:pg1232-DCN, F.Cu at (153.9, 96.8)
- added K13: diode-choc, pg1232:pg1232-DSS, F.Cu at (76.5, 93.2)
- added K14: diode-choc, pg1232:pg1232-DC, F.Cu at (89.0, 90.7)
- added K15: diode-choc, pg1232:pg1232-DC, F.Cu at (101.5, 88.2)
- added K16: diode-choc, pg1232:pg1232-DC, F.Cu at (118.7, 89.4)
- added K2: diode-choc, pg1232:pg1232-DC, F.Cu at (121.4, 35.1)
- added K3: diode-choc, pg1232:pg1232-DCL, F.Cu at (139.4, 42.1)
- added K4: diode-choc, pg1232:pg1232-DCN, F.Cu at (153.9, 71.8)
- added K5: diode-choc, pg1232:pg1232-DCR, F.Cu at (103.4, 54.6)
- added K6: diode-choc, pg1232:pg1232-DC, F.Cu at (121.4, 47.6)
- added K7: diode-choc, pg1232:pg1232-DCL, F.Cu at (139.4, 54.6)
- added K8: diode-choc, pg1232:pg1232-DCN, F.Cu at (153.9, 84.3)
- added K9: diode-choc, pg1232:pg1232-DCR, F.Cu at (103.4, 67.1)
- added L1: 10uH, Inductor_SMD:L_0603_1608Metric, F.Cu at (175.5, 83.6)
- added L2: 22uH, Inductor_SMD:L_Wuerth_WE-TPC-3816, F.Cu at (188.5, 17.2)
- added LCD1: adafruit-sharp-memory-display-no-useless, display:adafruit-sharp-memory-display-1.3in-no-mounting-no-useless, F.Cu at (140.9, 161.3)
- added Q1: AO3401A, Package_TO_SOT_SMD:SOT-23, F.Cu at (223.9, 67.7)
- added Q2: AO3400A, Package_TO_SOT_SMD:SOT-23, F.Cu at (227.3, 67.7)
- added R10: 5.1k, Resistor_SMD:R_0603_1608Metric, F.Cu at (233.9, 84.9)
- added R11: 22, Resistor_SMD:R_0603_1608Metric, F.Cu at (186.4, 68.7)
- added R12: 22, Resistor_SMD:R_0603_1608Metric, F.Cu at (224.1, 106.5)
- added R13: 4.12M, Resistor_SMD:R_0603_1608Metric, F.Cu at (187.5, 21.2)
- added R14: 10M, Resistor_SMD:R_0603_1608Metric, F.Cu at (184.5, 22.7)
- added R15: 5.9M, Resistor_SMD:R_0603_1608Metric, F.Cu at (187.5, 22.7)
- added R16: 5.1M, Resistor_SMD:R_0603_1608Metric, F.Cu at (190.5, 25.6)
- added R17: 5.1M, Resistor_SMD:R_0603_1608Metric, F.Cu at (190.5, 27.1)
- added R18: 5.1M, Resistor_SMD:R_0603_1608Metric, F.Cu at (194.0, 25.6)
- added R19: 5.1M, Resistor_SMD:R_0603_1608Metric, F.Cu at (194.0, 27.1)
- added R20: 1M, Resistor_SMD:R_0603_1608Metric, F.Cu at (195.3, 28.6)
- added R21: 4.12M, Resistor_SMD:R_0603_1608Metric, F.Cu at (196.8, 23.1)
- added R22: 4.87M, Resistor_SMD:R_0603_1608Metric, F.Cu at (196.8, 21.6)
- added R4: 1.2k, Resistor_SMD:R_0603_1608Metric, F.Cu at (218.3, 105.1)
- added R5: 1.5k, Resistor_SMD:R_0603_1608Metric, F.Cu at (219.8, 105.1)
- added R6: 1k, Resistor_SMD:R_0603_1608Metric, F.Cu at (221.3, 105.1)
- added R7: 1M, Resistor_SMD:R_0603_1608Metric, F.Cu at (233.8, 59.3)
- added R8: 10M, Resistor_SMD:R_0603_1608Metric, F.Cu at (228.9, 60.0)
- added R9: 5.1k, Resistor_SMD:R_0603_1608Metric, F.Cu at (219.9, 55.7)
- added REF**: jlc-tooling-hole, misc:jlc-tooling-hole, F.Cu at (211.6, 113.6)
- added REF**: nothing, misc:nothing, F.Cu at (156.0, 65.0)
- added REF**: nothing, misc:nothing, F.Cu at (173.0, 95.2)
- added REF**: jlc-tooling-hole, misc:jlc-tooling-hole, F.Cu at (211.3, 116.6)
- added SC1: Solar_Cell, misc:KXOB25-05X3F, F.Cu at (183.6, 38.6)
- added SW1: SW_Push, Button_Switch_SMD:SW_SPST_TL3342, F.Cu at (213.8, 47.0)
- added SW2: SW_SPDT, Button_Switch_SMD:SW_SPDT_PCM12, F.Cu at (199.5, 76.2)
- added U3: LN4913, Package_TO_SOT_SMD:SOT-23, F.Cu at (234.4, 68.2)
- added U4: XC6220B331MR, Package_TO_SOT_SMD:SOT-23-5, F.Cu at (222.4, 57.5)
- added U5: TLV70237_SOT23-5, Package_TO_SOT_SMD:SOT-23-5, F.Cu at (231.3, 63.5)
- added U6: SRV05-4, Package_TO_SOT_SMD:SOT-23-6, F.Cu at (187.0, 65.3)
- added U7: ~, Package_DFN_QFN:QFN-16-1EP_3x3mm_P0.5mm_EP1.7x1.7mm, F.Cu at (192.0, 21.9)
- J1: value Conn_01x04 -> debug-port; footprint steno:OLED -> misc:debug-port-single-side
- J2: value Conn_01x06 -> USB_C_Receptacle_USB2.0; footprint fistion:thumb-thumb -> Connector_USB:USB_C_Receptacle_HRO_TYPE-C-31-M-12
- R1: value 10k -> 100k; footprint Resistor_SMD:R_0805_2012Metric -> Resistor_SMD:R_0603_1608Metric; moved to F.Cu
- R2: value 10k -> 5.1M; footprint Resistor_SMD:R_0805_2012Metric -> Resistor_SMD:R_0603_1608Metric
- R3: value 10k -> 5.1M; footprint Resistor_SMD:R_0805_2012Metric -> Resistor_SMD:R_0603_1608Metric; moved to F.Cu
- U1: value nice_nano -> MT25QL128ABA1ESE; footprint nice-nano-kicad:nice_nano -> Package_SO:SOIC-8_5.23x5.23mm_P1.27mm
- U2: value MT25QL128ABA1ESE -> ms88sf3-nrf52840; footprint Package_SO:SOP-8_5.28x5.23mm_P1.27mm -> mcu:ms88sf3; moved to F.Cu
- moved J2 137.4 mm to (228.7, 53.0), turned to 60 degrees
- moved J1 136.0 mm to (213.9, 56.7), turned to 22.5 degrees
- moved R3 95.8 mm to (228.1, 76.2)
- moved U1 74.7 mm to (216.4, 94.8), turned to 90 degrees
- moved U2 44.5 mm to (175.6, 111.3), turned to -90 degrees
- moved R1 30.0 mm to (177.2, 79.7), turned to 0 degrees
- moved R2 23.3 mm to (171.5, 83.6), turned to 0 degrees
Connections:
- J1 pad 3: SCL -> /SWD
- J1 pad 4: SDA -> /SWC
- R1 pad 1: Net-(PUSH1-Pad1) -> 3V3
- R1 pad 2: 3V3 -> Net-(R1-Pad2)
- R2 pad 1: Net-(PUSH1-Pad1) -> /BAT
- R2 pad 2: 3V3 -> /BAT_MEAS
- R3 pad 1: 3V3 -> /BAT_MEAS
- R3 pad 2: Net-(R3-Pad2) -> GND
- U1 pad 1: SDA -> /FLASH_~{CS}
- U1 pad 2: SCL -> /MISO_DQ1
- U1 pad 3: GND -> Net-(R1-Pad2)
- U1 pad 5: CS -> /MOSI_DQ0
- U1 pad 6: MISO -> SCLK
- U1 pad 7: SCLK -> Net-(R1-Pad2)
- U1 pad 8: MOSI -> 3V3
- U2 pad 1: CS -> GND
- U2 pad 2: MISO -> unconnected-(U2-Pad2)
- U2 pad 3: Net-(R3-Pad2) -> unconnected-(U2-Pad3)
- U2 pad 4: GND -> unconnected-(U2-Pad4)
- U2 pad 5: MOSI -> unconnected-(U2-Pad5)
- U2 pad 6: SCLK -> unconnected-(U2-Pad6)
- U2 pad 7: Net-(R3-Pad2) -> unconnected-(U2-Pad7)
- U2 pad 8: 3V3 -> unconnected-(U2-Pad8)
Routing:
- net GND: track 319.1 -> 31.8 mm, vias 1 -> 4
- net /C0: track 0.00 -> 199.1 mm, vias 0 -> 1
- net 3V3: track 151.3 -> 0.00 mm
- net /C3: track 0.00 -> 140.2 mm
- net /C1: track 0.00 -> 128.1 mm
- net SDA: track 117.7 -> 0.00 mm, vias 1 -> 0
- net /R2: track 0.00 -> 108.0 mm
- net SCL: track 107.1 -> 0.00 mm, vias 1 -> 0
- net /C2: track 0.00 -> 98.6 mm, vias 0 -> 2
- net /R1: track 0.00 -> 95.1 mm
- net R1C3: track 95.0 -> 0.00 mm
- net /R0: track 0.00 -> 90.2 mm
- net R1C2: track 85.8 -> 0.00 mm
- net R1C4: track 77.4 -> 0.00 mm
- net R2C3: track 76.9 -> 0.00 mm
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- added copper zone on B.Cu, net GND
- added copper zone on F.Cu, net GND
Other:
- board outline removed
- net class Default removed
- board text removed: "JLCJLCJLCJLC"

Commit message: routed
Parts:
- removed D1: D_Small, Diode_SMD:D_SOD-123
- removed Q1: AO3401A, Package_TO_SOT_SMD:SOT-23
- removed Q2: AO3400A, Package_TO_SOT_SMD:SOT-23
- removed R7: 1M, Resistor_SMD:R_0603_1608Metric
- removed R8: 10M, Resistor_SMD:R_0603_1608Metric
- removed SW2: SW_SPDT, Button_Switch_SMD:SW_SPDT_PCM12
- added C10: 100nF, Capacitor_SMD:C_0603_1608Metric, F.Cu at (118.9, 92.2)
- added C11: 100nF, Capacitor_SMD:C_0603_1608Metric, F.Cu at (133.4, 87.5)
- added C12: 100uF, Capacitor_SMD:C_0603_1608Metric, F.Cu at (132.7, 90.5)
- added C13: 10nF, Capacitor_SMD:C_0603_1608Metric, F.Cu at (120.2, 80.7)
- added C14: 10uF, Capacitor_SMD:C_0603_1608Metric, F.Cu at (133.4, 95.5)
- added C15: 10nF, Capacitor_SMD:C_0603_1608Metric, F.Cu at (133.4, 97.0)
- added C9: 100nF, Capacitor_SMD:C_0603_1608Metric, F.Cu at (86.9, 76.7)
- added J10: Conn_01x06_Male, fistion:bridge, B.Cu at (7.20, 91.5)
- added J3: Conn_01x06_Male, fistion:bridge, B.Cu at (-64.8, 91.5)
- added J4: Conn_01x06_Male, fistion:bridge, B.Cu at (-30.8, 91.5)
- added J5: Conn_01x06_Male, fistion:bridge, B.Cu at (66.7, 90.7)
- added J6: Conn_01x06_Male, fistion:bridge, F.Cu at (-32.8, 91.5)
- added J7: Conn_01x06_Male, fistion:bridge, F.Cu at (39.2, 91.5)
- added J8: Conn_01x06_Male, fistion:bridge, F.Cu at (102.7, 90.7)
- added J9: Conn_01x06_Male, fistion:bridge, F.Cu at (5.20, 91.5)
- added U8: PMW3610, sensor:PMW3610, F.Cu at (125.7, 87.5)
- added U9: MCP1804x-1802xMB, Package_TO_SOT_SMD:SOT-89-3, F.Cu at (117.7, 76.7)
- C3: value 0.1uF -> 100nF
- JP2: value SolderJumper_3_Open -> jumper
- K16: moved to B.Cu
- SC1: value Solar_Cell -> solar
- U3: value LN4913 -> LSM6DS3; footprint Package_TO_SOT_SMD:SOT-23 -> Package_LGA:LGA-14_3x2.5mm_P0.5mm_LayoutBorder3x4y
- moved D2 239.9 mm to (-26.8, 97.7), turned to 0 degrees
- moved SC1 204.2 mm to (-13.6, 91.5), turned to 180 degrees
- moved REF** 169.1 mm to (47.2, 74.0)
- moved REF** 161.7 mm to (53.1, 83.0)
- moved U3 150.1 mm to (84.4, 75.2), turned to 0 degrees
- moved R6 149.6 mm to (72.9, 85.7), turned to 180 degrees
- moved R3 149.6 mm to (78.7, 82.0), turned to 180 degrees
- moved R10 149.1 mm to (88.7, 50.7)
- moved SW1 148.9 mm to (72.7, 94.5), turned to -90 degrees
- moved R5 148.0 mm to (72.9, 87.2), turned to 180 degrees
- moved C1 146.3 mm to (78.7, 83.5)
- moved R4 146.3 mm to (72.9, 88.7), turned to 180 degrees
- moved U1 139.7 mm to (77.9, 76.0), turned to 180 degrees
- moved J1 138.3 mm to (75.7, 52.0), turned to 45 degrees
- moved J2 137.8 mm to (91.2, 44.5), turned to 180 degrees
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Connections:
- net /3V3_LDO renamed 3V3_LDO
- net /BAT renamed BAT
- net /C1 renamed C1
- net /SWC renamed SWC
- net /SWD renamed SWD
- net /VBUS renamed VBUS
- C1 pad 1: /BAT_MEAS -> BAT_MEAS
- C2 pad 1: 3V3 -> 3V3_nRF
- C3 pad 1: /SOLAR_OUT -> 3V3_nRF
- C7 pad 2: /SOLAR_OUT -> SOLAR_OUT
- C8 pad 1: /SOLAR_OUT -> SOLAR_OUT
- D2 pad 2: 3V3 -> Net-(D2-Pad2)
- J1 pad 2: 3V3 -> 3V3_nRF
- J2 pad A6: /D+ -> D+
- J2 pad A7: /D- -> D-
- J2 pad B6: /D+ -> D+
- J2 pad B7: /D- -> D-
- JP1 pad 1: 3V3 -> 3V3_nRF
- JP1 pad 2: /VDDH -> SOLAR_OUT
- JP2 pad 1: /power/VDDH_EN -> SOLAR_OUT
- JP2 pad 3: /power/3V3_EN -> 3V3_nRF
- K1 pad 1: /R0 -> R0
- K1 pad 2: /C0 -> C0
- K10 pad 1: /R2 -> R2
- K11 pad 1: /R2 -> R2
- K11 pad 2: /C2 -> C2
- K12 pad 1: /R2 -> R2
- K12 pad 2: /C3 -> C3
- K13 pad 1: /R3 -> Net-(J3-Pad2)
- K13 pad 2: /C0 -> Net-(J3-Pad1)
- K14 pad 1: /R3 -> R3
- K15 pad 1: /R3 -> Net-(J10-Pad3)
- K15 pad 2: /C2 -> Net-(J10-Pad1)
- K16 pad 1: /R3 -> Net-(J9-Pad3)
- K16 pad 2: /C3 -> Net-(J9-Pad2)
- K2 pad 1: /R0 -> R0
- K3 pad 1: /R0 -> R0
- K3 pad 2: /C2 -> C2
- K4 pad 1: /R0 -> R0
- K4 pad 2: /C3 -> C3
- K5 pad 1: /R1 -> R1
- K5 pad 2: /C0 -> C0
- K6 pad 1: /R1 -> R1
- K7 pad 1: /R1 -> R1
- K7 pad 2: /C2 -> C2
- K8 pad 1: /R1 -> R1
- K8 pad 2: /C3 -> C3
- K9 pad 1: /R2 -> R2
- K9 pad 2: /C0 -> C0
- L1 pad 2: 3V3 -> 3V3_nRF
- LCD1 pad 5: 3V3 -> 3V3_nRF
- R1 pad 1: 3V3 -> 3V3_nRF
- R2 pad 2: /BAT_MEAS -> BAT_MEAS
- R3 pad 1: /BAT_MEAS -> BAT_MEAS
- R4 pad 1: /~{RED} -> ~{RED}
- R4 pad 2: Net-(D2-Pad1) -> Net-(J5-Pad5)
- R5 pad 1: /~{GREEN} -> ~{GREEN}
- R5 pad 2: Net-(D2-Pad4) -> Net-(J5-Pad4)
- R6 pad 1: /~{BLUE} -> ~{BLUE}
- R6 pad 2: Net-(D2-Pad3) -> Net-(J5-Pad3)
- SC1 pad 1: /power/SOLAR -> Net-(J9-Pad5)
- SC1 pad 2: GND -> Net-(J9-Pad6)
- U1 pad 1: /FLASH_~{CS} -> FLASH_~{CS}
- U1 pad 2: /MISO_DQ1 -> MISO_DQ1
- U1 pad 5: /MOSI_DQ0 -> MOSI_DQ0
- U1 pad 8: 3V3 -> 3V3_nRF
- U2 pad 10: /~{RED} -> unconnected-(U2-Pad10)
- U2 pad 11: /~{GREEN} -> unconnected-(U2-Pad11)
- U2 pad 12: /~{BLUE} -> unconnected-(U2-Pad12)
- U2 pad 14: unconnected-(U2-Pad14) -> FLASH_~{CS}
- U2 pad 15: unconnected-(U2-Pad15) -> MISO_DQ1
- U2 pad 16: /BAT_MEAS -> MOSI_DQ0
- U2 pad 17: unconnected-(U2-Pad17) -> SCLK
- U2 pad 19: /R3 -> IMU_~{CS}
- U2 pad 2: unconnected-(U2-Pad2) -> ~{BLUE}
- U2 pad 20: /MID_BTN -> IMU_INT
- U2 pad 21: /IR_EN -> DISP_~{CS}
- U2 pad 22: /ENC_OUT -> unconnected-(U2-Pad22)
- U2 pad 23: /TP_~{CS} -> MOTION
- U2 pad 24: /TP_DR -> MOUSE_~{RST}
- U2 pad 25: /MISO_DQ1 -> MOUSE_~{CS}
- U2 pad 26: /FLASH_~{CS} -> SCLK2
- U2 pad 27: /MOSI_DQ0 -> SDIO
- U2 pad 29: SCLK -> unconnected-(U2-Pad29)
- U2 pad 3: unconnected-(U2-Pad3) -> ~{GREEN}
- U2 pad 31: 3V3 -> 3V3_nRF
- U2 pad 32: /VDDH -> SOLAR_OUT
- U2 pad 36: /D- -> D-
- U2 pad 37: /D+ -> D+
- U2 pad 38: DISP_~{CS} -> unconnected-(U2-Pad38)
- U2 pad 39: /IO_~{CS} -> unconnected-(U2-Pad39)
- U2 pad 4: unconnected-(U2-Pad4) -> ~{RED}
- U2 pad 40: /IO_INT -> unconnected-(U2-Pad40)
- U2 pad 41: /C0_LEFT -> R3
- U2 pad 42: /R1 -> R2
- U2 pad 43: /R0 -> R1
- U2 pad 44: /C4 -> R0
- U2 pad 45: /C3 -> C3
- U2 pad 46: /C2 -> C2
- U2 pad 48: /C0 -> C0
- U2 pad 60: Net-(D1-Pad1) -> unconnected-(U2-Pad60)
- U2 pad 9: /R2 -> BAT_MEAS
- U3 pad 1: /SOLAR_OUT -> MISO_DQ1
- U3 pad 2: /MAGNET -> GND
- U4 pad 1: /SOLAR_OUT -> SOLAR_OUT
- U4 pad 3: /power/3V3_EN -> SOLAR_OUT
- U6 pad 1: /D- -> D+
- U6 pad 3: /D+ -> D-
- U6 pad 4: /D+ -> D-
- U6 pad 6: /D- -> D+
- U7 pad 15: /SOLAR_OUT -> SOLAR_OUT
Routing:
- net /C0: track 199.1 -> 0.00 mm, vias 1 -> 0
- net C2: track 0.00 -> 168.1 mm, vias 0 -> 1
- net /C3: track 140.2 -> 0.00 mm
- net C3: track 0.00 -> 139.3 mm, vias 0 -> 1
- net 3V3_nRF: track 0.00 -> 130.6 mm, vias 0 -> 4
- net /R2: track 108.0 -> 0.00 mm
- net C0: track 0.00 -> 104.7 mm, vias 0 -> 4
- net /C2: track 98.6 -> 0.00 mm, vias 2 -> 0
- net /R1: track 95.1 -> 0.00 mm
- net R2: track 0.00 -> 94.1 mm, vias 0 -> 1
- net R1: track 0.00 -> 93.9 mm, vias 0 -> 1
- net R0: track 0.00 -> 91.9 mm, vias 0 -> 1
- net /R0: track 90.2 -> 0.00 mm
- net BAT: track 1.24 -> 85.6 mm, vias 1 -> 3
- net R3: track 0.00 -> 73.5 mm, vias 0 -> 1
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Other:
- board outline added: 226 x 66.2 mm
- board text added: "- solar & LED goes on top (top thumb?) - screen may go on top/left side"
