File: musk.kicad_pcb (KiCad board)
At the start: 2 copper layers, 106 x 104 mm, 97 parts, among them J1 debug-port, J10 bridge, J2 USB_C_Receptacle_USB2.0, J3 bridge, J4 bridge, J5 bridge, J6 bridge, J7 bridge, J8 bridge, J9 bridge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

Commit message: fabed
Parts:
- moved J10 3.00 mm to (134.0, 21.0)
- moved J3 3.00 mm to (54.0, 21.0)
- moved J6 3.00 mm to (86.0, 21.0)
- moved J7 3.00 mm to (166.0, 21.0)
- moved K15 3.00 mm to (145.7, 21.0)
- moved SW1 3.00 mm to (70.0, 21.0)
Routing:
- net GND: track 67.9 -> 84.4 mm
Other:
- board size 106 x 104 mm -> 112 x 104 mm
